File: hamilton-thermostat-main.brd (EAGLE design)
At the start: 88.9 x 61 mm, 128 parts, among them J1 TC2030-JLINK-NL, J2 PHOENIX6W5MM, K1_G TX2S2SA-L2-3V, K2_Y TX2S2SA-L2-3V, K3_W TX2S2SA-L2-3V, Q1 MMBT2222A, Q2 MMBT2222A, Q3 MMBT2222A, Q4 MMBT2222A, Q5 MMBT2222A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

Commit message: Move relay jumper location
Parts:
- moved R17 16.1 mm to (32.3, 35.8), turned to 180 degrees
- moved U7 3.94 mm to (36.6, 27.9)
- moved R18 3.43 mm to (32.3, 37.1), turned to 180 degrees
Routing:
- net N$50: track 5.91 -> 21.9 mm
- net PIRSIG: track 74.9 -> 70.9 mm
- net N$51: track 6.54 -> 9.09 mm
- net R: track 100.3 -> 101.4 mm, vias 1 -> 3
Changed lines of the file:
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@@
 <layer number="17" name="Pads" color="2" fill="1" visible="yes" active="yes"/>
 <layer number="18" name="Vias" color="2" fill="1" visible="yes" active="yes"/>
-<layer number="19" name="Unrouted" color="6" fill="1" visible="no" active="yes"/>
+<layer number="19" name="Unrouted" color="6" fill="1" visible="yes" active="yes"/>
 <layer number="20" name="Dimension" color="15" fill="1" visible="yes" active="yes"/>
 <layer number="21" name="tPlace" color="7" fill="1" visible="yes" active="yes"/>
@@
 <attribute name="NAME" x="6.263" y="4.112" size="1.016" layer="25" font="vector"/>
 </element>
-<element name="U7" library="storm" package="PIR" value="PANASONIC_PIR" x="36.576" y="31.877" smashed="yes" rot="R270">
-<attribute name="NAME" x="35.052" y="26.543" size="1.016" layer="25" font="vector" rot="R180"/>
+<element name="U7" library="storm" package="PIR" value="PANASONIC_PIR" x="36.576" y="27.94" smashed="yes" rot="R270">
+<attribute name="NAME" x="35.052" y="22.606" size="1.016" layer="25" font="vector" rot="R180"/>
 </element>
 <element name="U6" library="storm" package="SOT23" value="SOT23-3VREG" x="55.753" y="25.4" smashed="yes" rot="R180">
@@
 <attribute name="VALUE" x="24.843" y="11.6205" size="1.016" layer="27" font="vector" ratio="12" rot="R270" align="bottom-center"/>
 </element>
-<element name="R17" library="storm" package="S0402" value="0R" x="16.256" y="37.084" smashed="yes" rot="R90">
-<attribute name="NAME" x="15.7099" y="36.3093" size="1.016" layer="25" rot="R90"/>
-</element>
-<element name="R18" library="storm" package="S0402" value="0R" x="28.829" y="37.084" smashed="yes" rot="R90">
-<attribute name="NAME" x="28.2829" y="36.3093" size="1.016" layer="25" font="vector" rot="R90"/>
+<element name="R17" library="storm" package="S0402" value="0R" x="32.258" y="35.814" smashed="yes" rot="R180">
+<attribute name="NAME" x="30.861" y="36.322" size="1.016" layer="25" rot="R180"/>
+</element>
+<element name="R18" library="storm" package="S0402" value="0R" x="32.258" y="37.1475" smashed="yes" rot="R180">
+<attribute name="NAME" x="30.861" y="37.719" size="1.016" layer="25" font="vector" rot="R180"/>
 </element>
 <element name="C30" library="storm" package="0805" value="10uF" x="55.753" y="28.829" smashed="yes" rot="R180">
@@
 <via x="40.132" y="17.018" extent="1-16" drill="0.3048"/>
 <wire x1="40.386" y1="13.081" x2="40.386" y2="16.764" width="0.1524" layer="1"/>
-<wire x1="34.036" y1="29.337" x2="34.036" y2="20.574" width="0.1524" layer="16"/>
+<wire x1="34.036" y1="25.4" x2="34.036" y2="20.574" width="0.1524" layer="16"/>
 </signal>
 <signal name="N$15">
@@
 <contactref element="D9" pad="A"/>
 <wire x1="6.667" y1="42.164" x2="1.969" y2="42.164" width="0.4064" layer="1"/>
-<wire x1="28.829" y1="36.068" x2="36.83" y2="36.068" width="0.4064" layer="1"/>
 <contactref element="R17" pad="P$1"/>
 <contactref element="R18" pad="P$1"/>
-<wire x1="28.829" y1="36.068" x2="22.098" y2="36.068" width="0.4064" layer="1"/>
-<wire x1="22.098" y1="36.068" x2="16.256" y2="36.068" width="0.4064" layer="1"/>
-<wire x1="28.829" y1="36.068" x2="28.829" y2="37.084" width="0.4064" layer="1"/>
-<wire x1="16.256" y1="36.068" x2="12.7" y2="36.068" width="0.4064" layer="1"/>
+<wire x1="12.7" y1="36.068" x2="22.098" y2="36.068" width="0.4064" layer="1"/>
 <wire x1="12.7" y1="36.068" x2="10.16" y2="38.608" width="0.4064" layer="1"/>
 <wire x1="10.16" y1="38.608" x2="10.16" y2="41.021" width="0.4064" layer="1"/>
 <wire x1="10.16" y1="41.021" x2="9.017" y2="42.164" width="0.4064" layer="1"/>
 <wire x1="9.017" y1="42.164" x2="6.667" y2="42.164" width="0.4064" layer="1"/>
-<wire x1="16.256" y1="36.068" x2="16.256" y2="37.084" width="0.4064" layer="1"/>
-<wire x1="22.098" y1="36.068" x2="22.098" y2="40.894" width="0.4064" layer="1"/>
-<wire x1="22.098" y1="40.894" x2="20.828" y2="42.164" width="0.4064" layer="1"/>
+<wire x1="20.828" y1="42.164" x2="22.098" y2="40.894" width="0.4064" layer="1"/>
 <wire x1="20.828" y1="42.164" x2="18.605" y2="42.164" width="0.4064" layer="1"/>
 <wire x1="43.57" y1="47.371" x2="41.647" y2="47.371" width="0.4064" layer="1"/>
-<wire x1="36.83" y1="36.068" x2="40.386" y2="39.624" width="0.4064" layer="1"/>
 <wire x1="40.386" y1="39.624" x2="40.386" y2="46.237" width="0.4064" layer="1"/>
 <wire x1="40.386" y1="46.237" x2="41.647" y2="47.371" width="0.4064" layer="1"/>
@@
 <wire x1="71.12" y1="38.26" x2="71.12" y2="40.767" width="0.4064" layer="16"/>
 <wire x1="71.12" y1="40.767" x2="69.85" y2="42.037" width="0.4064" layer="16"/>
+<via x="22.098" y="40.894" extent="1-16" drill="0.6096"/>
+<via x="22.098" y="36.068" extent="1-16" drill="0.6096"/>
+<wire x1="22.098" y1="36.068" x2="27.7495" y2="36.068" width="0.4064" layer="1"/>
+<wire x1="27.7495" y1="36.068" x2="28.8925" y2="34.925" width="0.4064" layer="1"/>
+<wire x1="22.098" y1="36.068" x2="22.098" y2="40.894" width="0.4064" layer="16"/>
+<wire x1="32.258" y1="34.925" x2="28.8925" y2="34.925" width="0.4064" layer="1"/>
+<wire x1="32.258" y1="34.925" x2="35.687" y2="34.925" width="0.4064" layer="1"/>
+<wire x1="35.687" y1="34.925" x2="40.386" y2="39.624" width="0.4064" layer="1"/>
+<wire x1="32.258" y1="35.814" x2="32.258" y2="34.925" width="0.4064" layer="1"/>
+<wire x1="32.258" y1="35.814" x2="32.258" y2="37.1475" width="0.4064" layer="1"/>
 </signal>
 <signal name="Y">
@@
 <contactref element="R17" pad="P$2"/>
 <contactref element="K2_Y" pad="4"/>
-<wire x1="16.256" y1="37.934" x2="16.256" y2="41.021" width="0.4064" layer="1"/>
 <wire x1="16.256" y1="41.021" x2="15.113" y2="42.164" width="0.4064" layer="1"/>
 <wire x1="15.113" y1="42.164" x2="13.907" y2="42.164" width="0.4064" layer="1"/>
+<wire x1="16.8275" y1="37.465" x2="16.256" y2="38.0365" width="0.4064" layer="1"/>
+<wire x1="16.256" y1="38.0365" x2="16.256" y2="41.021" width="0.4064" layer="1"/>
+<wire x1="28.448" y1="37.465" x2="16.8275" y2="37.465" width="0.4064" layer="1"/>
+<wire x1="31.408" y1="35.814" x2="30.099" y2="35.814" width="0.4064" layer="1"/>
+<wire x1="30.099" y1="35.814" x2="28.448" y2="37.465" width="0.4064" layer="1"/>
 </signal>
 <signal name="N$51">
 <contactref element="R18" pad="P$2"/>
 <contactref element="K3_W" pad="4"/>
-<wire x1="28.829" y1="37.934" x2="28.829" y2="41.021" width="0.4064" layer="1"/>
 <wire x1="28.829" y1="41.021" x2="27.813" y2="42.037" width="0.4064" layer="1"/>
 <wire x1="27.813" y1="42.037" x2="25.972" y2="42.037" width="0.4064" layer="1"/>
 <wire x1="25.972" y1="42.037" x2="25.845" y2="42.164" width="0.4064" layer="1"/>
+<wire x1="31.408" y1="37.1475" x2="30.226" y2="37.1475" width="0.4064" layer="1"/>
+<wire x1="30.226" y1="37.1475" x2="28.829" y2="38.5445" width="0.4064" layer="1"/>
+<wire x1="28.829" y1="38.5445" x2="28.829" y2="41.021" width="0.4064" layer="1"/>
 </signal>
 </signals>
